File: hardware/sensors/v2/sensors.sch (EAGLE design)
At the start: 38 parts, among them IC1 MEGA8-AI, IC3 7805TV, IC4 MAX232ECWE

Commit message: changes to fix a bug in the hardware and make it DRC proof
Connections:
- removed net N$21: R8.2, U$1./RESET
- removed net N$29: IC1.ADC6, JP8.1
- new net /CANRST: IC1.ADC6, JP8.1, R8.2, U$1./RESET
- net MISO: now also U$1.SO; no longer U$1.SI
- net MOSI: now also U$1.SI; no longer U$1.SO
Other:
- moved on the sheet: R8
Changed lines of the file:
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@@
 <instance part="P+13" gate="VCC" x="99.06" y="33.02" rot="R270"/>
 <instance part="GND17" gate="1" x="215.9" y="73.66" rot="R180"/>
-<instance part="R8" gate="G$1" x="220.98" y="58.42" rot="R180"/>
+<instance part="R8" gate="G$1" x="226.06" y="58.42" rot="R180"/>
 <instance part="P+14" gate="VCC" x="236.22" y="58.42" rot="R270"/>
 <instance part="C7" gate="G$1" x="215.9" y="66.04"/>
@@
 <pinref part="R8" gate="G$1" pin="1"/>
 <pinref part="P+14" gate="VCC" pin="VCC"/>
-<wire x1="233.68" y1="58.42" x2="226.06" y2="58.42" width="0.1524" layer="91"/>
+<wire x1="233.68" y1="58.42" x2="231.14" y2="58.42" width="0.1524" layer="91"/>
 </segment>
 <segment>
@@
 <net name="MOSI" class="0">
 <segment>
-<pinref part="U$1" gate="G$1" pin="SO"/>
-<wire x1="213.36" y1="53.34" x2="233.68" y2="53.34" width="0.1524" layer="91"/>
-<label x="223.52" y="53.34" size="1.778" layer="95"/>
-</segment>
-<segment>
 <wire x1="40.64" y1="7.62" x2="86.36" y2="7.62" width="0.1524" layer="91"/>
 <label x="78.74" y="7.62" size="1.778" layer="95"/>
@@
 <label x="111.76" y="-20.32" size="1.778" layer="95" rot="R90"/>
 </segment>
-</net>
-<net name="MISO" class="0">
 <segment>
 <pinref part="U$1" gate="G$1" pin="SI"/>
@@
 <label x="223.52" y="50.8" size="1.778" layer="95"/>
 </segment>
+</net>
+<net name="MISO" class="0">
 <segment>
 <wire x1="40.64" y1="5.08" x2="86.36" y2="5.08" width="0.1524" layer="91"/>
@@
 <wire x1="121.92" y1="-5.08" x2="121.92" y2="-20.32" width="0.1524" layer="91"/>
 <label x="121.92" y="-20.32" size="1.778" layer="95" rot="R90"/>
+</segment>
+<segment>
+<pinref part="U$1" gate="G$1" pin="SO"/>
+<wire x1="233.68" y1="53.34" x2="213.36" y2="53.34" width="0.1524" layer="91"/>
+<label x="223.52" y="53.34" size="1.778" layer="95"/>
 </segment>
 </net>
@@
 </segment>
 </net>
-<net name="N$21" class="0">
+<net name="/CANRST" class="0">
 <segment>
 <pinref part="R8" gate="G$1" pin="2"/>
 <pinref part="U$1" gate="G$1" pin="/RESET"/>
-<wire x1="215.9" y1="58.42" x2="213.36" y2="58.42" width="0.1524" layer="91"/>
+<wire x1="220.98" y1="58.42" x2="213.36" y2="58.42" width="0.1524" layer="91"/>
+<label x="215.9" y="58.42" size="1.778" layer="95"/>
+</segment>
+<segment>
+<pinref part="IC1" gate="G$1" pin="ADC6"/>
+<wire x1="40.64" y1="45.72" x2="48.26" y2="45.72" width="0.1524" layer="91"/>
+<wire x1="48.26" y1="45.72" x2="48.26" y2="43.18" width="0.1524" layer="91"/>
+<wire x1="48.26" y1="43.18" x2="71.12" y2="43.18" width="0.1524" layer="91"/>
+<wire x1="71.12" y1="43.18" x2="71.12" y2="48.26" width="0.1524" layer="91"/>
+<pinref part="JP8" gate="A" pin="1"/>
+<wire x1="71.12" y1="48.26" x2="86.36" y2="48.26" width="0.1524" layer="91"/>
+<label x="50.8" y="43.18" size="1.778" layer="95"/>
 </segment>
 </net>
@@
 </segment>
 </net>
-<net name="N$29" class="0">
-<segment>
-<pinref part="IC1" gate="G$1" pin="ADC6"/>
-<wire x1="40.64" y1="45.72" x2="48.26" y2="45.72" width="0.1524" layer="91"/>
-<wire x1="48.26" y1="45.72" x2="48.26" y2="43.18" width="0.1524" layer="91"/>
-<wire x1="48.26" y1="43.18" x2="71.12" y2="43.18" width="0.1524" layer="91"/>
-<wire x1="71.12" y1="43.18" x2="71.12" y2="48.26" width="0.1524" layer="91"/>
-<pinref part="JP8" gate="A" pin="1"/>
-<wire x1="71.12" y1="48.26" x2="86.36" y2="48.26" width="0.1524" layer="91"/>
-</segment>
-</net>
